Commit message: Create config file for wx250s arm in curobo

File: src/curobo/content/assets/robot/widowx/wx250s.urdf (robot description, URDF)
Before this commit: robot wx250s, 14 links, 13 joints
Links:
- removed link wx250s/base_link
- removed link wx250s/ee_arm_link
- removed link wx250s/ee_gripper_link
- removed link wx250s/fingers_link
- removed link wx250s/gripper_bar_link
- removed link wx250s/gripper_link
- removed link wx250s/gripper_prop_link
- removed link wx250s/left_finger_link
- removed link wx250s/lower_forearm_link
- removed link wx250s/right_finger_link
- removed link wx250s/shoulder_link
- removed link wx250s/upper_arm_link
- removed link wx250s/upper_forearm_link
- removed link wx250s/wrist_link
- added link base_link, mass 0.538736; collision mesh filename=meshes/wx250s_1_base.stl; visual mesh filename=meshes/wx250s_1_base.stl
- added link ee_arm_link, mass 0.001
- added link ee_gripper_link, mass 0.001
- added link fingers_link, mass 0.001
- added link gripper_bar_link, mass 0.034199; collision mesh filename=meshes/wx250s_9_gripper_bar.stl; visual mesh filename=meshes/wx250s_9_gripper_bar.stl
- added link gripper_link, mass 0.072885; collision mesh filename=meshes/wx250s_7_gripper.stl; visual mesh filename=meshes/wx250s_7_gripper.stl
- added link gripper_prop_link, mass 0.00434; collision mesh filename=meshes/wx250s_8_gripper_prop.stl; visual mesh filename=meshes/wx250s_8_gripper_prop.stl
- added link left_finger_link, mass 0.016246; collision mesh filename=meshes/wx250s_10_gripper_finger.stl; visual mesh filename=meshes/wx250s_10_gripper_finger.stl
- added link lower_forearm_link, mass 0.220991; collision mesh filename=meshes/wx250s_5_lower_forearm.stl; visual mesh filename=meshes/wx250s_5_lower_forearm.stl
- added link right_finger_link, mass 0.016246; collision mesh filename=meshes/wx250s_10_gripper_finger.stl; visual mesh filename=meshes/wx250s_10_gripper_finger.stl
- added link shoulder_link, mass 0.480879; collision mesh filename=meshes/wx250s_2_shoulder.stl; visual mesh filename=meshes/wx250s_2_shoulder.stl
- added link upper_arm_link, mass 0.430811; collision mesh filename=meshes/wx250s_3_upper_arm.stl; visual mesh filename=meshes/wx250s_3_upper_arm.stl
- added link upper_forearm_link, mass 0.234589; collision mesh filename=meshes/wx250s_4_upper_forearm.stl; visual mesh filename=meshes/wx250s_4_upper_forearm.stl
- added link wrist_link, mass 0.084957; collision mesh filename=meshes/wx250s_6_wrist.stl; visual mesh filename=meshes/wx250s_6_wrist.stl
Joints:
- joint ee_arm: child wx250s/ee_arm_link -> ee_arm_link; parent wx250s/gripper_link -> gripper_link
- joint ee_bar: child wx250s/fingers_link -> fingers_link; parent wx250s/gripper_bar_link -> gripper_bar_link
- joint ee_gripper: child wx250s/ee_gripper_link -> ee_gripper_link; parent wx250s/fingers_link -> fingers_link
- joint forearm_roll: child wx250s/lower_forearm_link -> lower_forearm_link; parent wx250s/upper_forearm_link -> upper_forearm_link
- joint gripper: child wx250s/gripper_prop_link -> gripper_prop_link; parent wx250s/ee_arm_link -> ee_arm_link
- joint gripper_bar: child wx250s/gripper_bar_link -> gripper_bar_link; parent wx250s/ee_arm_link -> ee_arm_link
- joint widow_elbow: child wx250s/upper_forearm_link -> upper_forearm_link; parent wx250s/upper_arm_link -> upper_arm_link
- joint widow_left_finger: child wx250s/left_finger_link -> left_finger_link; parent wx250s/fingers_link -> fingers_link
- joint widow_right_finger: child wx250s/right_finger_link -> right_finger_link; parent wx250s/fingers_link -> fingers_link
- joint widow_shoulder: child wx250s/upper_arm_link -> upper_arm_link; parent wx250s/shoulder_link -> shoulder_link
- joint widow_waist: child wx250s/shoulder_link -> shoulder_link; limit effort=10 velocity=3.141592653589793 -> lower=-3.141582653589793 upper=3.141582653589793 effort=10 velocity=3.141592653589793; parent wx250s/base_link -> base_link
- joint widow_wrist_angle: child wx250s/wrist_link -> wrist_link; parent wx250s/lower_forearm_link -> lower_forearm_link
- joint widow_wrist_rotate: child wx250s/gripper_link -> gripper_link; parent wx250s/wrist_link -> wrist_link
