Commit message: Separate actual URDF from URDF with fake prismatic joints used by curobo

File: src/curobo/content/assets/robot/sagittarius/K1Go1_curobo.urdf (robot description, URDF)
Before this commit: robot K1Go1, 34 links, 33 joints
Links:
- added link mobile_base_link_tx
- added link mobile_base_link_ty
- added link mobile_base_link_yaw
Joints:
- added joint mobile_base_tx: type prismatic, parent base, child mobile_base_link_tx, origin xyz=0 0 0.0 rpy=0 0 0.0, axis 1 0 0, limit lower=-10.0 upper=10.0 effort=87 velocity=0.5
- added joint mobile_base_ty: type prismatic, parent mobile_base_link_tx, child mobile_base_link_ty, origin xyz=0 0 0.0 rpy=0 0 0.0, axis 0 1 0, limit lower=-10.0 upper=10.0 effort=87 velocity=0.5
- added joint mobile_base_yaw: type revolute, parent mobile_base_link_ty, child mobile_base_link_yaw, origin xyz=0 0 0.0 rpy=0 0 0.0, axis 0 0 1, limit lower=-6.0 upper=6.0 effort=87 velocity=1.50
- joint floating_base: origin xyz=0 0 0.0 rpy=0 0 0.0 -> xyz=0 0 0.45 rpy=0 0 0.0; parent base -> mobile_base_link_yaw
